File: blinky_PCB/blinky_PCB.kicad_pcb (KiCad board)
At the start: 2 copper layers, 40 x 30 mm, 7 parts, among them J1 Barrel_Jack_MountingPin, U1 NE555P

Commit message: updated PCB cam
Parts:
- moved J1 0.75 mm to (119.0, 87.5)
Routing:
- net +9V: track 35.5 -> 36.0 mm
